Commit message: Fix VR buttons and update lift range

File: software/lerobot-hei-rebot-lift/examples/hei_rebot_lift/VR_mujoco_ik/mujoco_ik/model/HEI_robot_urdf/urdf/HEI_robot_urdf.urdf (robot description, URDF)
Before this commit: robot HEI_robot_urdf, 38 links, 37 joints
Joints:
- joint lift_joint: limit lower=-0.8 upper=0 effort=0 velocity=0 -> lower=-0.7 upper=0 effort=0 velocity=0
